File: hardware/arpie_cv_tab.brd (EAGLE design)
At the start: 35.9 x 57.2 mm, 62 parts, among them IC1 MCP4726, IC2 MCP601OT, IC3 LM27675M5_CHARGEPUMP, IC4 LM358D, IC5 LM4041A12DBZ

Commit message: v5 added eeprom
Parts:
- removed C11: (no value), rcl:E2,5-5
- added C12: (no value), resistor:C0805
- added IC6: 24LC_16BT-I/OT, Microchip-24LCxxx:SOT95P290X145-5N
- CLK_LED, GATE_LED: device adafruit:LED3MM -> led:CHIP-LED0805
- moved GATE_LED 0.38 mm to (88.9, 16.1), turned to 0 degrees
- turned CLK_LED to 0 degrees
- turned R10 to 270 degrees
Connections:
- net +5V: now also C12.2, IC6.4; no longer C11.+
- net GND: now also C12.1, IC6.2, IC6.5; no longer C11.-
- net N$2: now also CLK_LED.C; no longer CLK_LED.K
- net N$3: now also GATE_LED.C; no longer GATE_LED.K
- net SCL: now also IC6.1
- net SDA: now also IC6.3
Routing:
- net SDA: track 52.6 -> 75.7 mm, vias 2 -> 4
- net SCL: track 49.3 -> 71.9 mm, vias 2 -> 4
- net GND: track 63.0 -> 68.7 mm, vias 12 -> 13
- net +5V: track 92.5 -> 96.8 mm
- net N$1: track 24.8 -> 20.9 mm
- net N$3: track 5.52 -> 4.49 mm
- net N$9: track 24.1 -> 24.6 mm
Other:
- board text added: "CLK"
- board text added: "GATE"
- board text added: "V4"
- board text removed: "V3"
