File: hardware/arpie_cv_tab.sch (EAGLE design)
At the start: 63 parts, among them IC1 MCP4726, IC2 MCP601OT, IC3 LM27675M5_CHARGEPUMP, IC4 LM358D, IC5 LM4041A12DBZ, IC6 24LC_16BT-I/OT

Commit message: add values to schematic
Parts:
- R11, R8: value (none) -> 2m2
- R4, R5: value (none) -> 1k
- R6: value 100k -> 47k
- R7: value (none) -> 47k
Changed lines of the file:
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@@
 <part name="C5" library="resistor" deviceset="C-EU" device="C0805"/>
 <part name="C4" library="resistor" deviceset="C-EU" device="C0805"/>
-<part name="R5" library="rcl" deviceset="R-EU_" device="R0805"/>
+<part name="R5" library="rcl" deviceset="R-EU_" device="R0805" value="1k"/>
 <part name="GND16" library="SparkFun" deviceset="GND" device=""/>
-<part name="R4" library="rcl" deviceset="R-EU_" device="R0805"/>
+<part name="R4" library="rcl" deviceset="R-EU_" device="R0805" value="1k"/>
 <part name="SUPPLY1" library="supply2" deviceset="+5V" device=""/>
 <part name="GND7" library="SparkFun" deviceset="GND" device=""/>
@@
 <part name="SUPPLY7" library="supply2" deviceset="+10V" device=""/>
 <part name="IC4" library="linear" deviceset="LM358" device="D"/>
-<part name="R7" library="rcl" deviceset="R-EU_" device="R0805"/>
-<part name="R6" library="rcl" deviceset="R-EU_" device="R0805" value="100k"/>
+<part name="R7" library="rcl" deviceset="R-EU_" device="R0805" value="47k"/>
+<part name="R6" library="rcl" deviceset="R-EU_" device="R0805" value="47k"/>
 <part name="GND11" library="SparkFun" deviceset="GND" device=""/>
 <part name="SUPPLY2" library="supply2" deviceset="+5V" device=""/>
@@
 <part name="R12" library="rcl" deviceset="R-EU_" device="R0805" value="100k"/>
 <part name="R9" library="rcl" deviceset="R-EU_" device="R0805" value="100k"/>
-<part name="R8" library="rcl" deviceset="R-EU_" device="R0805"/>
-<part name="R11" library="rcl" deviceset="R-EU_" device="R0805"/>
+<part name="R8" library="rcl" deviceset="R-EU_" device="R0805" value="2m2"/>
+<part name="R11" library="rcl" deviceset="R-EU_" device="R0805" value="2m2"/>
 <part name="C10" library="resistor" deviceset="C-EU" device="C0805"/>
 <part name="IC5" library="texas" deviceset="LM4041" device="DBZ" technology="A12"/>

Commit message: V5 - change type of 3.5mm socket
Parts:
- CLKOUT, CVOUT, GATEOUT: value SMD35MMJACK -> 3_5MM_PTH_MICRO; device jasons_stuff:SMD35MMJACK -> jason_eagle6:3_5MM_PTH_MICRO
Connections:
- net CVOUT: now also CVOUT.4; no longer CVOUT.T
- net GND: now also CLKOUT.2, CLKOUT.3, CVOUT.2, CVOUT.3, GATEOUT.2, GATEOUT.3; no longer CLKOUT.R, CLKOUT.S, CVOUT.R, CVOUT.S, GATEOUT.R, GATEOUT.S
- net N$19: now also CLKOUT.4; no longer CLKOUT.T
- net N$20: now also GATEOUT.4; no longer GATEOUT.T
Other:
- note added: "VERSION 5 - 28jan18"
- note removed: "VERSION 4 - 18dec18"
Changed lines of the file:
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@@
 <part name="SUPPLY4" library="supply2" deviceset="+5V" device=""/>
 <part name="GND13" library="SparkFun" deviceset="GND" device=""/>
-<part name="CLKOUT" library="jasons_stuff" deviceset="SMD35MMJACK" device=""/>
-<part name="GATEOUT" library="jasons_stuff" deviceset="SMD35MMJACK" device=""/>
-<part name="CVOUT" library="jasons_stuff" deviceset="SMD35MMJACK" device=""/>
 <part name="IC1" library="jasons_stuff" deviceset="MCP4726" device=""/>
 <part name="C5" library="resistor" deviceset="C-EU" device="C0805"/>
@@
 <part name="C12" library="resistor" deviceset="C-EU" device="C0805"/>
 <part name="GND26" library="SparkFun" deviceset="GND" device=""/>
+<part name="CLKOUT" library="jason_eagle6" deviceset="3_5MM_PTH_MICRO" device=""/>
+<part name="GATEOUT" library="jason_eagle6" deviceset="3_5MM_PTH_MICRO" device=""/>
+<part name="CVOUT" library="jason_eagle6" deviceset="3_5MM_PTH_MICRO" device=""/>
 </parts>
 <sheets>
@@
 <text x="193.04" y="19.05" size="3.81" layer="91">&amp; LEVEL SHIFTER</text>
 <text x="58.166" y="26.67" size="5.08" layer="91">CV TAB FOR ARPIE</text>
-<text x="58.42" y="20.32" size="5.08" layer="91">VERSION 4 - 18dec18</text>
+<text x="58.42" y="20.32" size="5.08" layer="91">VERSION 5 - 28jan18</text>
 <text x="58.42" y="12.7" size="3.81" layer="91">Sixty four pixels limited</text>
 <text x="58.42" y="7.62" size="3.81" layer="91">CC-NC-BY-SA Not to be used for commercial purposes</text>
@@
 <instance part="SUPPLY4" gate="+5V" x="114.3" y="185.42"/>
 <instance part="GND13" gate="1" x="147.32" y="160.02"/>
-<instance part="CLKOUT" gate="G$1" x="276.86" y="86.36" rot="R270"/>
-<instance part="GATEOUT" gate="G$1" x="276.86" y="60.96" rot="R270"/>
-<instance part="CVOUT" gate="G$1" x="276.86" y="35.56" rot="R270"/>
 <instance part="IC1" gate="G$1" x="96.52" y="127"/>
 <instance part="C5" gate="G$1" x="254" y="81.28"/>
@@
 <instance part="C12" gate="G$1" x="162.56" y="142.24" rot="R180"/>
 <instance part="GND26" gate="1" x="162.56" y="124.46"/>
+<instance part="CLKOUT" gate="G$1" x="289.56" y="86.36" rot="R180"/>
+<instance part="GATEOUT" gate="G$1" x="289.56" y="60.96" rot="R180"/>
+<instance part="CVOUT" gate="G$1" x="289.56" y="35.56" rot="R180"/>
 </instances>
 <busses>
@@
 </segment>
 <segment>
-<pinref part="CLKOUT" gate="G$1" pin="S"/>
-<wire x1="271.78" y1="91.44" x2="266.7" y2="91.44" width="0.1524" layer="91"/>
-<wire x1="266.7" y1="91.44" x2="266.7" y2="81.28" width="0.1524" layer="91"/>
-<pinref part="CLKOUT" gate="G$1" pin="R"/>
-<wire x1="266.7" y1="81.28" x2="266.7" y2="71.12" width="0.1524" layer="91"/>
-<wire x1="266.7" y1="71.12" x2="266.7" y2="66.04" width="0.1524" layer="91"/>
-<wire x1="266.7" y1="66.04" x2="266.7" y2="55.88" width="0.1524" layer="91"/>
-<wire x1="271.78" y1="81.28" x2="266.7" y2="81.28" width="0.1524" layer="91"/>
-<junction x="266.7" y="81.28"/>
-<pinref part="GATEOUT" gate="G$1" pin="S"/>
-<wire x1="271.78" y1="66.04" x2="266.7" y2="66.04" width="0.1524" layer="91"/>
-<junction x="266.7" y="66.04"/>
-<pinref part="GATEOUT" gate="G$1" pin="R"/>
-<wire x1="271.78" y1="55.88" x2="266.7" y2="55.88" width="0.1524" layer="91"/>
-<junction x="266.7" y="55.88"/>
-<wire x1="266.7" y1="55.88" x2="266.7" y2="45.72" width="0.1524" layer="91"/>
-<pinref part="CVOUT" gate="G$1" pin="S"/>
-<wire x1="266.7" y1="45.72" x2="266.7" y2="40.64" width="0.1524" layer="91"/>
-<wire x1="266.7" y1="40.64" x2="266.7" y2="30.48" width="0.1524" layer="91"/>
-<wire x1="266.7" y1="30.48" x2="266.7" y2="25.4" width="0.1524" layer="91"/>
-<wire x1="271.78" y1="40.64" x2="266.7" y2="40.64" width="0.1524" layer="91"/>
-<junction x="266.7" y="40.64"/>
-<pinref part="CVOUT" gate="G$1" pin="R"/>
-<wire x1="271.78" y1="30.48" x2="266.7" y2="30.48" width="0.1524" layer="91"/>
-<junction x="266.7" y="30.48"/>
+<wire x1="266.7" y1="88.9" x2="266.7" y2="83.82" width="0.1524" layer="91"/>
+<wire x1="266.7" y1="83.82" x2="266.7" y2="71.12" width="0.1524" layer="91"/>
+<wire x1="266.7" y1="71.12" x2="266.7" y2="63.5" width="0.1524" layer="91"/>
+<wire x1="266.7" y1="63.5" x2="266.7" y2="58.42" width="0.1524" layer="91"/>
+<junction x="266.7" y="83.82"/>
+<junction x="266.7" y="63.5"/>
+<junction x="266.7" y="58.42"/>
+<wire x1="266.7" y1="58.42" x2="266.7" y2="45.72" width="0.1524" layer="91"/>
+<wire x1="266.7" y1="45.72" x2="266.7" y2="38.1" width="0.1524" layer="91"/>
+<wire x1="266.7" y1="38.1" x2="266.7" y2="33.02" width="0.1524" layer="91"/>
+<wire x1="266.7" y1="33.02" x2="266.7" y2="25.4" width="0.1524" layer="91"/>
+<junction x="266.7" y="38.1"/>
+<junction x="266.7" y="33.02"/>
 <pinref part="GND16" gate="1" pin="GND"/>
 <pinref part="C4" gate="G$1" pin="2"/>
@@
 <wire x1="254" y1="71.12" x2="266.7" y2="71.12" width="0.1524" layer="91"/>
 <junction x="266.7" y="71.12"/>
+<pinref part="CVOUT" gate="G$1" pin="3"/>
+<wire x1="266.7" y1="38.1" x2="279.4" y2="38.1" width="0.1524" layer="91"/>
+<pinref part="CVOUT" gate="G$1" pin="2"/>
+<wire x1="266.7" y1="33.02" x2="279.4" y2="33.02" width="0.1524" layer="91"/>
+<pinref part="CLKOUT" gate="G$1" pin="3"/>
+<wire x1="279.4" y1="88.9" x2="266.7" y2="88.9" width="0.1524" layer="91"/>
+<pinref part="CLKOUT" gate="G$1" pin="2"/>
+<wire x1="266.7" y1="83.82" x2="279.4" y2="83.82" width="0.1524" layer="91"/>
+<pinref part="GATEOUT" gate="G$1" pin="3"/>
+<wire x1="266.7" y1="63.5" x2="279.4" y2="63.5" width="0.1524" layer="91"/>
+<pinref part="GATEOUT" gate="G$1" pin="2"/>
+<wire x1="266.7" y1="58.42" x2="279.4" y2="58.42" width="0.1524" layer="91"/>
 </segment>
 <segment>
@@
 <segment>
 <pinref part="R5" gate="G$1" pin="2"/>
-<pinref part="CLKOUT" gate="G$1" pin="T"/>
 <wire x1="248.92" y1="86.36" x2="254" y2="86.36" width="0.1524" layer="91"/>
 <pinref part="C5" gate="G$1" pin="1"/>
-<wire x1="254" y1="86.36" x2="271.78" y2="86.36" width="0.1524" layer="91"/>
+<wire x1="254" y1="86.36" x2="279.4" y2="86.36" width="0.1524" layer="91"/>
 <wire x1="254" y1="83.82" x2="254" y2="86.36" width="0.1524" layer="91"/>
 <junction x="254" y="86.36"/>
+<pinref part="CLKOUT" gate="G$1" pin="4"/>
 </segment>
 </net>
@@
 <segment>
 <pinref part="R4" gate="G$1" pin="2"/>
-<pinref part="GATEOUT" gate="G$1" pin="T"/>
 <wire x1="248.92" y1="60.96" x2="254" y2="60.96" width="0.1524" layer="91"/>
 <pinref part="C4" gate="G$1" pin="1"/>
-<wire x1="254" y1="60.96" x2="271.78" y2="60.96" width="0.1524" layer="91"/>
+<wire x1="254" y1="60.96" x2="279.4" y2="60.96" width="0.1524" layer="91"/>
 <wire x1="254" y1="58.42" x2="254" y2="60.96" width="0.1524" layer="91"/>
 <junction x="254" y="60.96"/>
+<pinref part="GATEOUT" gate="G$1" pin="4"/>
 </segment>
 </net>
@@
 </segment>
 <segment>
-<pinref part="CVOUT" gate="G$1" pin="T"/>
-<wire x1="271.78" y1="35.56" x2="246.38" y2="35.56" width="0.1524" layer="91"/>
 <label x="236.22" y="35.56" size="1.778" layer="95"/>
-</segment>
-</net>
+<pinref part="CVOUT" gate="G$1" pin="4"/>
+<wire x1="246.38" y1="35.56" x2="279.4" y2="35.56" width="0.1524" layer="91"/>
+</segment>
+</net>
